Commit message: Complete ROS 2 AgroBot: collision-aware tasks, four scenarios, README
- Task layer: box collision model built from the URDF, joint-space
  RRT-Connect planner, collision-checked IK and linear moves, rail used as
  an external axis with reachability checks, crops and fixtures as obstacles
- New scenarios: seedling transplanting, precision weeding and plant
  inspection, alongside strawberry harvesting; per-run KPI reports
- Robot model: split base/gripper collision boxes, raised crate beside the
  arm, camera mast moved out of the arm's reach, inline material colours,
  collision-free home pose, rail starting off its end stop
- Worlds: static crop fixtures (joints to world froze the rail in Fortress),
  soil blocks in a shallow tray, weeds and tray rows inside the top-down
  workspace
- Unit tests for kinematics, collision checking and planning
- README: architecture, scenarios with simulation results, and step-by-step
  instructions for commissioning the real robot

File: aibomech_agrobot_description/urdf/agrobot.urdf.xacro (robot description, xacro)
@@ -17,6 +17,6 @@
   <xacro:arg name="use_camera" default="true"/>
   <!-- Camera pose relative to arm_mount: "x y z" and "roll pitch yaw" -->
-  <xacro:arg name="camera_xyz" default="0.0 -0.15 0.60"/>
-  <xacro:arg name="camera_rpy" default="0 1.0 1.5708"/>
+  <xacro:arg name="camera_xyz" default="-0.20 -0.18 0.60"/>
+  <xacro:arg name="camera_rpy" default="0 0.93 1.075"/>
   <xacro:arg name="initial_positions_file" default="$(find aibomech_agrobot_description)/config/initial_positions.yaml"/>
   <xacro:arg name="calibration_file" default="$(find aibomech_agrobot_description)/config/hardware_calibration.yaml"/>
@@ -51,5 +51,6 @@
   <xacro:if value="$(arg use_camera)">
     <xacro:rgbd_camera prefix="${prefix}" parent="${prefix}arm_mount" xyz="$(arg camera_xyz)" rpy="$(arg camera_rpy)"
-                       mast_height="${float('$(arg camera_xyz)'.split()[2]) + 0.02}" sim="${hardware == 'gz'}"/>
+                       mast_height="${float('$(arg camera_xyz)'.split()[2]) + 0.02}" sim="${hardware == 'gz'}"
+                       mast_bottom="${-(float('$(arg mount_height)') - 0.455) if platform == 'rail_trolley' else 0.0}"/>
   </xacro:if>
   <xacro:agrobot_ros2_control prefix="${prefix}" hardware="${hardware}" use_rail="${use_rail}"

File: aibomech_agrobot_description/urdf/arm.xacro (robot description, xacro)
@@ -35,9 +35,13 @@
           <mesh filename="${mesh_dir}/${name}.STL"/>
         </geometry>
-        <material name="${material}"/>
+        <xacro:mat name="${material}"/>
       </visual>
       <xacro:arm_collision_box box="${p['collision_box']}"/>
       <xacro:if value="${'collision_box_jaw' in p}">
         <xacro:arm_collision_box box="${p['collision_box_jaw']}"/>
+      </xacro:if>
+      <xacro:if value="${'collision_box_post' in p}">
+        <xacro:arm_collision_box box="${p['collision_box_post']}"/>
+        <xacro:arm_collision_box box="${p['collision_box_bracket']}"/>
       </xacro:if>
     </link>

File: aibomech_agrobot_description/urdf/camera.xacro (robot description, xacro)
@@ -7,14 +7,16 @@
 -->
 <robot xmlns:xacro="http://www.ros.org/wiki/xacro">
-  <xacro:macro name="rgbd_camera" params="prefix parent xyz rpy mast_height sim">
+  <xacro:macro name="rgbd_camera" params="prefix parent xyz rpy mast_height sim mast_bottom:=0.0">
+    <!-- The mast runs from mast_bottom (e.g. the cabinet lid) to the camera. -->
+    <xacro:property name="mast_len" value="${mast_height - mast_bottom}"/>
     <link name="${prefix}camera_mast">
       <visual>
-        <origin xyz="0 0 ${mast_height/2}" rpy="0 0 0"/>
-        <geometry><box size="0.02 0.02 ${mast_height}"/></geometry>
-        <material name="aluminium"/>
+        <origin xyz="0 0 ${mast_bottom + mast_len/2}" rpy="0 0 0"/>
+        <geometry><box size="0.02 0.02 ${mast_len}"/></geometry>
+        <xacro:mat name="aluminium"/>
       </visual>
       <collision>
-        <origin xyz="0 0 ${mast_height/2}" rpy="0 0 0"/>
-        <geometry><box size="0.02 0.02 ${mast_height}"/></geometry>
+        <origin xyz="0 0 ${mast_bottom + mast_len/2}" rpy="0 0 0"/>
+        <geometry><box size="0.02 0.02 ${mast_len}"/></geometry>
       </collision>
       <inertial>
@@ -33,5 +35,5 @@
         <origin xyz="-0.0125 0 0" rpy="0 0 0"/>
         <geometry><box size="0.025 0.09 0.025"/></geometry>
-        <material name="black"/>
+        <xacro:mat name="black"/>
       </visual>
       <collision>

File: aibomech_agrobot_description/urdf/materials.xacro (robot description, xacro)
@@ -1,13 +1,20 @@
 <?xml version="1.0"?>
+<!-- Colours. Visuals use <xacro:mat name="..."/> so every material carries its
+     colour inline: Gazebo drops named-only materials on links merged by
+     fixed-joint reduction and renders them black. -->
 <robot xmlns:xacro="http://www.ros.org/wiki/xacro">
-  <material name="agro_orange"><color rgba="0.93 0.45 0.07 1"/></material>
-  <material name="graphite"><color rgba="0.20 0.21 0.23 1"/></material>
-  <material name="aluminium"><color rgba="0.76 0.77 0.79 1"/></material>
-  <material name="cabinet_grey"><color rgba="0.60 0.62 0.64 1"/></material>
-  <material name="black"><color rgba="0.06 0.06 0.06 1"/></material>
-  <material name="pipe_white"><color rgba="0.92 0.92 0.90 1"/></material>
-  <material name="crate_green"><color rgba="0.10 0.45 0.20 1"/></material>
-  <material name="safety_yellow"><color rgba="1.00 0.80 0.00 1"/></material>
-  <material name="estop_red"><color rgba="0.85 0.05 0.05 1"/></material>
-  <material name="signal_green"><color rgba="0.10 0.85 0.20 1"/></material>
+  <xacro:property name="agro_colors" value="${dict(
+      agro_orange='0.93 0.45 0.07 1',
+      graphite='0.20 0.21 0.23 1',
+      aluminium='0.76 0.77 0.79 1',
+      cabinet_grey='0.60 0.62 0.64 1',
+      black='0.06 0.06 0.06 1',
+      pipe_white='0.92 0.92 0.90 1',
+      crate_green='0.10 0.45 0.20 1',
+      safety_yellow='1.00 0.80 0.00 1',
+      estop_red='0.85 0.05 0.05 1',
+      signal_green='0.10 0.85 0.20 1')}"/>
+  <xacro:macro name="mat" params="name">
+    <material name="${name}"><color rgba="${agro_colors[name]}"/></material>
+  </xacro:macro>
 </robot>

File: aibomech_agrobot_description/urdf/platform.xacro (robot description, xacro)
@@ -30,5 +30,5 @@
       <origin xyz="${xyz}" rpy="0 0 0"/>
       <geometry><box size="${size}"/></geometry>
-      <material name="${material}"/>
+      <xacro:mat name="${material}"/>
     </visual>
     <xacro:if value="${collision}">
@@ -43,5 +43,5 @@
       <origin xyz="${x} ${y} ${rail_height + rail_pipe_radius + 0.02}" rpy="${pi/2} 0 0"/>
       <geometry><cylinder radius="0.045" length="0.03"/></geometry>
-      <material name="black"/>
+      <xacro:mat name="black"/>
     </visual>
   </xacro:macro>
@@ -50,6 +50,9 @@
   <xacro:macro name="lift_column" params="prefix parent base_z mount_height crate">
     <xacro:property name="col_len" value="${mount_height - base_z - 0.01}"/>
-    <!-- crate floor 88 mm below the mounting plate -->
-    <xacro:property name="crate_z" value="${col_len - 0.078}"/>
+    <!-- Crate floor 40 mm below the mounting plate, on a bracket at +x: at the
+         arm's height, so carried crops never swing under the mounting plate. -->
+    <xacro:property name="crate_z" value="${col_len - 0.03}"/>
+    <xacro:property name="crate_x" value="0.26"/>
+    <xacro:property name="crate_y" value="-0.04"/>
     <link name="${prefix}lift_column">
       <xacro:box_inertial mass="6.0" x="${column_size}" y="${column_size}" z="${col_len}">
@@ -57,14 +60,13 @@
       </xacro:box_inertial>
       <xacro:box_part name="column" size="${column_size} ${column_size} ${col_len}" xyz="0 0 ${col_len/2}" material="aluminium"/>
-      <xacro:box_part name="top_plate" size="0.20 0.22 0.01" xyz="0 -0.04 ${col_len + 0.005}" material="graphite"/>
+      <xacro:box_part name="top_plate" size="0.12 0.12 0.01" xyz="0 0 ${col_len + 0.005}" material="graphite"/>
       <xacro:if value="${crate}">
-        <!-- Harvest crate on a shelf beside the arm (+x), inside its reach and
-             outside the camera's view of the crop row. -->
-        <xacro:box_part name="shelf" size="0.26 0.14 0.008" xyz="0.17 -0.08 ${crate_z - 0.006}" material="aluminium"/>
-        <xacro:box_part name="crate_floor" size="0.16 0.12 0.004" xyz="0.20 -0.08 ${crate_z}" material="crate_green"/>
-        <xacro:box_part name="crate_wall_n" size="0.16 0.004 0.045" xyz="0.20 -0.022 ${crate_z + 0.0245}" material="crate_green"/>
-        <xacro:box_part name="crate_wall_s" size="0.16 0.004 0.045" xyz="0.20 -0.138 ${crate_z + 0.0245}" material="crate_green"/>
-        <xacro:box_part name="crate_wall_e" size="0.004 0.12 0.045" xyz="0.278 -0.08 ${crate_z + 0.0245}" material="crate_green"/>
-        <xacro:box_part name="crate_wall_w" size="0.004 0.12 0.045" xyz="0.122 -0.08 ${crate_z + 0.0245}" material="crate_green"/>
+        <xacro:box_part name="crate_bracket" size="0.12 0.03 0.008" xyz="0.10 ${crate_y} ${crate_z - 0.006}" material="aluminium"/>
+        <xacro:box_part name="shelf" size="0.20 0.14 0.008" xyz="${crate_x} ${crate_y} ${crate_z - 0.006}" material="aluminium"/>
+        <xacro:box_part name="crate_floor" size="0.16 0.12 0.004" xyz="${crate_x} ${crate_y} ${crate_z}" material="crate_green"/>
+        <xacro:box_part name="crate_wall_n" size="0.16 0.004 0.045" xyz="${crate_x} ${crate_y + 0.058} ${crate_z + 0.0245}" material="crate_green"/>
+        <xacro:box_part name="crate_wall_s" size="0.16 0.004 0.045" xyz="${crate_x} ${crate_y - 0.058} ${crate_z + 0.0245}" material="crate_green"/>
+        <xacro:box_part name="crate_wall_e" size="0.004 0.12 0.045" xyz="${crate_x + 0.078} ${crate_y} ${crate_z + 0.0245}" material="crate_green"/>
+        <xacro:box_part name="crate_wall_w" size="0.004 0.12 0.045" xyz="${crate_x - 0.078} ${crate_y} ${crate_z + 0.0245}" material="crate_green"/>
       </xacro:if>
     </link>
@@ -84,5 +86,5 @@
       <link name="${prefix}crate"/>
       <joint name="${prefix}crate_joint" type="fixed">
-        <origin xyz="0.20 -0.08 ${crate_z + 0.002}" rpy="0 0 0"/>
+        <origin xyz="${crate_x} ${crate_y} ${crate_z + 0.002}" rpy="0 0 0"/>
         <parent link="${prefix}lift_column"/>
         <child link="${prefix}crate"/>
@@ -101,10 +103,10 @@
         <origin xyz="${rail_x} ${rail_gauge/2} ${rail_height}" rpy="0 ${pi/2} 0"/>
         <geometry><cylinder radius="${rail_pipe_radius}" length="${pipe_len}"/></geometry>
-        <material name="pipe_white"/>
+        <xacro:mat name="pipe_white"/>
       </visual>
       <visual name="pipe_right">
         <origin xyz="${rail_x} ${-rail_gauge/2} ${rail_height}" rpy="0 ${pi/2} 0"/>
         <geometry><cylinder radius="${rail_pipe_radius}" length="${pipe_len}"/></geometry>
-        <material name="pipe_white"/>
+        <xacro:mat name="pipe_white"/>
       </visual>
     </link>
@@ -126,16 +128,16 @@
         <origin xyz="-0.12 -0.10 ${deck_z + deck_thickness/2 + 0.255}" rpy="0 0 0"/>
         <geometry><box size="0.07 0.07 0.03"/></geometry>
-        <material name="safety_yellow"/>
+        <xacro:mat name="safety_yellow"/>
       </visual>
       <visual name="estop_button">
         <origin xyz="-0.12 -0.10 ${deck_z + deck_thickness/2 + 0.28}" rpy="0 0 0"/>
         <geometry><cylinder radius="0.02" length="0.02"/></geometry>
-        <material name="estop_red"/>
+        <xacro:mat name="estop_red"/>
       </visual>
       <!-- Signal tower -->
       <visual name="signal_tower">
-        <origin xyz="-0.21 -0.17 ${deck_z + deck_thickness/2 + 0.30}" rpy="0 0 0"/>
+        <origin xyz="-0.04 -0.16 ${deck_z + deck_thickness/2 + 0.30}" rpy="0 0 0"/>
         <geometry><cylinder radius="0.012" length="0.12"/></geometry>
-        <material name="signal_green"/>
+        <xacro:mat name="signal_green"/>
       </visual>
       <!-- Flanged wheels riding on the pipes -->
