Commit message: Enhance collision detection and handling for precision weeding and seedling transplant tasks
- Updated the CollisionModel to include an obstacle clearance parameter, ensuring that obstacles remain a safe distance away from the robot's held objects.
- Modified the RobotInterface to incorporate held object dimensions and offsets for improved collision checking during movement.
- Refactored the PrecisionWeeding task to include a retry mechanism for weed removal attempts, logging outcomes and distances to nearby crops.
- Added configuration parameters for held object sizes and offsets in both precision weeding and seedling transplant YAML files, allowing for better collision detection with the robot's gripper.

File: agrobot_ws/src/aibomech_agrobot_description/urdf/arm.xacro (robot description, xacro)
@@ -21,4 +21,6 @@
   <xacro:property name="tcp_y" value="0.0725"/>
   <xacro:property name="tcp_z" value="-0.008"/>
+  <!-- Middle between the fixed jaw face (-0.016) and the open moving jaw (+0.009) -->
+  <xacro:property name="tcp_center_z" value="-0.003"/>
   <xacro:macro name="arm_link" params="prefix name material">
     <xacro:property name="p" value="${arm_phys[name]}"/>
@@ -118,4 +120,12 @@
       <child link="${prefix}tcp"/>
     </joint>
+    <!-- tcp_center: middle of the open jaw gap. Use it for thin objects (stems)
+         that must not touch the fixed jaw on the way in. -->
+    <link name="${prefix}tcp_center"/>
+    <joint name="${prefix}link_4-tcp_center" type="fixed">
+      <origin xyz="${tcp_x} ${tcp_y} ${tcp_center_z}" rpy="0 ${-pi/2} 0"/>
+      <parent link="${prefix}link_4"/>
+      <child link="${prefix}tcp_center"/>
+    </joint>
   </xacro:macro>
 </robot>

File: agrobot_ws/src/aibomech_agrobot_tasks/test/data/agrobot.urdf (robot description, URDF)
Before this commit: robot agrobot, 19 links, 18 joints
Links:
- added link tcp_center
Joints:
- added joint link_4-tcp_center: type fixed, parent link_4, child tcp_center, origin xyz=-0.135 0.0725 -0.003 rpy=0 -1.5707963267948966 0
